File: cmoy-nioh.kicad_pcb (KiCad board)
At the start: 2 copper layers, 72.9 x 58.6 mm, 14 parts, among them U1 OPA2604A

Commit message: 25.08.2017
Routing:
- net (no net): track 0.00 -> 44.4 mm
Changed lines of the file:
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@@
     (thickness 1.6)
     (drawings 5)
-    (tracks 100)
+    (tracks 101)
     (zones 0)
     (modules 14)
@@
   (gr_line (start 83.7 123) (end 156.6 123) (angle 90) (layer Edge.Cuts) (width 0.1))
   (gr_line (start 156.5 68) (end 156.5 123) (angle 90) (layer Edge.Cuts) (width 0.1))
+  (segment (start 95.25 92.71) (end 139.7 92.71) (width 0.5) (layer B.Cu) (net 0))
   (segment (start 104.16 119) (end 104.16 119.64) (width 0.7) (layer B.Cu) (net 1))
   (segment (start 112.4 67.4) (end 118.5 67.4) (width 0.7) (layer B.Cu) (net 1))

Commit message: z androida
Routing:
- net (no net): track 44.4 -> 87.6 mm
Changed lines of the file:
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@@
     (thickness 1.6)
     (drawings 5)
-    (tracks 101)
+    (tracks 102)
     (zones 0)
     (modules 14)
@@
   (gr_line (start 83.7 123) (end 156.6 123) (angle 90) (layer Edge.Cuts) (width 0.1))
   (gr_line (start 156.5 68) (end 156.5 123) (angle 90) (layer Edge.Cuts) (width 0.1))
+  (segment (start 96.52 95.25) (end 139.7 95.25) (width 0.5) (layer B.Cu) (net 0))
   (segment (start 95.25 92.71) (end 139.7 92.71) (width 0.5) (layer B.Cu) (net 0))
   (segment (start 104.16 119) (end 104.16 119.64) (width 0.7) (layer B.Cu) (net 1))
